File: KiCad-Files/rc_hotwheels.kicad_pcb (KiCad board)
At the start: 2 copper layers, 0 parts

Commit message: Created PCB Design
 - Placed Components at the right place. Connected Voltage Regulator chip to MCU.
- Changed Capacitors Footprint and Symbol.
Parts:
- added ?: , , F.Cu at (132.9, 71.1)
- added ?: , , F.Cu at (106.2, 74.2)
- added ?: , , F.Cu at (132.9, 76.2)
- added ?: , , F.Cu at (106.2, 71.6)
- added ?: , , F.Cu at (132.9, 73.7)
- added ?: , , B.Cu at (114.3, 66.0)
- added ?: , , B.Cu at (109.2, 66.0)
- added ?: , , B.Cu at (111.8, 66.0)
- added ?: , , B.Cu at (116.8, 66.0)
- added C1: 1uF, C1uF:CAPC1005X55N, F.Cu at (101.1, 63.5)
- added C2: 1uF, C1uF:CAPC1005X55N, F.Cu at (125.2, 69.1)
- added C3: 4.7uF, C4.7uF:CAPC1608X87N, F.Cu at (123.0, 63.1)
- added C3: 4.7uF, C4.7uF:CAPC1608X87N, F.Cu at (119.0, 61.7)
- added C4: 1uF, C1uF:CAPC1005X55N, F.Cu at (101.1, 66.0)
- added C5: 100nF, C100nF:CAPC1005X55N, F.Cu at (119.0, 63.2)
- added C5: 100nF, C100nF:CAPC1005X55N, F.Cu at (121.4, 63.2)
- added C6: 10nF, C10nF:CAPC1005X55N, F.Cu at (101.1, 68.6)
- added IC1: BD6211F-E2, BD6211F-E2:SOIC127P620X171-8N, F.Cu at (111.7, 73.1)
- added IC2: MIC5504-3.3YM5-TR, MIC5504-3.3YM5-TR:SOT95P280X145-5N, F.Cu at (126.0, 72.4)
- added S1: OS102011MS2QN1, OS102011MS2QN1:OS102011MA1QN1, F.Cu at (132.1, 82.1)
- added U1: STM32F070F6P6, STM32F070F6P6:SOP65P640X120-20N, F.Cu at (119.0, 73.1)
- added U3: NRF24L01_Breakout, RF_Module:nRF24L01_Breakout, F.Cu at (132.9, 62.2)
Routing:
- net VR_OUT: track 0.00 -> 49.0 mm, vias 0 -> 1
- net VCC: track 0.00 -> 31.9 mm
- net GND: track 0.00 -> 31.1 mm, vias 0 -> 3
- net VREF: track 0.00 -> 26.5 mm
- net RIN: track 0.00 -> 9.32 mm
- net Motor -: track 0.00 -> 7.44 mm
- net SYS_SWCLK: track 0.00 -> 4.84 mm
- net SYS_SWDIO: track 0.00 -> 4.59 mm
Other:
- board outline added: 30 x 26 mm
